Commit message: all namespaces are active

File: ros2_ws/src/panda_ign_description/urdf/panda_sim.urdf.xacro (robot description, xacro)
@@ -1,4 +1,7 @@
 <?xml version="1.0"?>
 <robot xmlns:xacro="http://www.ros.org/wiki/xacro" name="panda">
+  <!-- Xacro arguments -->
+  <xacro:arg name="namespace" default=""/>
+  <xacro:arg name="controller_config" default="$(find panda_ign_description)/config/panda_controllers.yaml"/>
   <!-- Include the base panda URDF -->
   <xacro:include filename="$(find panda_ign_description)/panda/panda.urdf"/>
@@ -89,5 +92,11 @@
   <gazebo>
     <plugin filename="libgz_ros2_control-system.so" name="gz_ros2_control::GazeboSimROS2ControlPlugin">
-      <parameters>$(find panda_ign_description)/config/panda_controllers.yaml</parameters>
+      <parameters>$(arg controller_config)</parameters>
+      <xacro:property name="ns" value="$(arg namespace)"/>
+      <xacro:if value="${len(ns) > 0}">
+        <ros>
+          <namespace>${ns}</namespace>
+        </ros>
+      </xacro:if>
     </plugin>
   </gazebo>
