Commit message: now transitioning to 1 controller, last insertion left

File: ros2_ws/src/panda_ign_description/panda/panda.urdf (robot description, URDF)
Before this commit: robot panda, 14 links, 13 joints
Links:
- added link panda_rightfinger_mimic, mass 1e-06
Joints:
- added joint panda_finger_joint2_mimic: type prismatic, parent panda_hand, child panda_rightfinger_mimic, origin xyz=0 0 0.0584 rpy=0 0 0, axis 0 -1 0, limit lower=-0.001 upper=0.04 effort=20. velocity=0.3, mimic joint=panda_finger_joint1
